File: BSPD.sch (KiCad schematic (older format))
At the start: 45 parts, among them J1 Conn_02x04_Odd_Even, J2 Screw_Terminal_01x02, K1 RT444012, Q1 IRLML2502, U1 AZ1117-5.0, U2 LM2901, U3 LM2901

Commit message: update schematics
Change regulator to ZLDO1117
Parts:
- U1: value AZ1117-5.0 -> ZLDO1117G50; footprint Package_TO_SOT_SMD:SOT-223 -> Package_TO_SOT_SMD:SOT-223-3_TabPin2; symbol Regulator_Linear:AZ1117-5.0 -> Regulator_Linear:AP1117-50
- U2, U3: value LM2901 -> LM2901D
Changed lines of the file:
@@
 EESchema Schematic File Version 4
-LIBS:BSPD-cache
 EELAYER 30 0
 EELAYER END
@@
 Date "2019-11-14"
 Rev "A"
-Comp "Oxford University Racing"
+Comp ""
 Comment1 ""
 Comment2 ""
@@
 P 3500 2400
 F 0 "U2" H 3500 2767 50  0000 C CNN
-F 1 "LM2901" H 3500 2676 50  0000 C CNN
+F 1 "LM2901D" H 3500 2676 50  0000 C CNN
 F 2 "Package_SO:SOIC-14_3.9x8.7mm_P1.27mm" H 3450 2500 50  0001 C CNN
 F 3 "~" H 3550 2600 50  0001 C CNN
@@
 P 3500 1500
 F 0 "U2" H 3500 1867 50  0000 C CNN
-F 1 "LM2901" H 3500 1776 50  0000 C CNN
+F 1 "LM2901D" H 3500 1776 50  0000 C CNN
 F 2 "Package_SO:SOIC-14_3.9x8.7mm_P1.27mm" H 3450 1600 50  0001 C CNN
 F 3 "~" H 3550 1700 50  0001 C CNN
@@
 P 3500 4700
 F 0 "U2" H 3500 5067 50  0000 C CNN
-F 1 "LM2901" H 3500 4976 50  0000 C CNN
+F 1 "LM2901D" H 3500 4976 50  0000 C CNN
 F 2 "Package_SO:SOIC-14_3.9x8.7mm_P1.27mm" H 3450 4800 50  0001 C CNN
 F 3 "~" H 3550 4900 50  0001 C CNN
@@
 P 5100 2300
 F 0 "U3" H 5100 2667 50  0000 C CNN
-F 1 "LM2901" H 5100 2576 50  0000 C CNN
+F 1 "LM2901D" H 5100 2576 50  0000 C CNN
 F 2 "Package_SO:SOIC-14_3.9x8.7mm_P1.27mm" H 5050 2400 50  0001 C CNN
 F 3 "~" H 5150 2500 50  0001 C CNN
@@
 P 3500 3800
 F 0 "U2" H 3500 4167 50  0000 C CNN
-F 1 "LM2901" H 3500 4076 50  0000 C CNN
+F 1 "LM2901D" H 3500 4076 50  0000 C CNN
 F 2 "Package_SO:SOIC-14_3.9x8.7mm_P1.27mm" H 3450 3900 50  0001 C CNN
 F 3 "~" H 3550 4000 50  0001 C CNN
@@
 P 7000 3100
 F 0 "U3" H 7000 3467 50  0000 C CNN
-F 1 "LM2901" H 7000 3376 50  0000 C CNN
+F 1 "LM2901D" H 7000 3376 50  0000 C CNN
 F 2 "Package_SO:SOIC-14_3.9x8.7mm_P1.27mm" H 6950 3200 50  0001 C CNN
 F 3 "~" H 7050 3300 50  0001 C CNN
@@
 P 3900 7000
 F 0 "U2" H 3858 7046 50  0000 L CNN
-F 1 "LM2901" H 3858 6955 50  0000 L CNN
+F 1 "LM2901D" H 3858 6955 50  0000 L CNN
 F 2 "Package_SO:SOIC-14_3.9x8.7mm_P1.27mm" H 3850 7100 50  0001 C CNN
 F 3 "~" H 3950 7200 50  0001 C CNN
@@
 P 4400 7000
 F 0 "U3" H 4358 7046 50  0000 L CNN
-F 1 "LM2901" H 4358 6955 50  0000 L CNN
+F 1 "LM2901D" H 4358 6955 50  0000 L CNN
 F 2 "Package_SO:SOIC-14_3.9x8.7mm_P1.27mm" H 4350 7100 50  0001 C CNN
 F 3 "~" H 4450 7200 50  0001 C CNN
@@
 Connection ~ 4300 7300
 $Comp
-L Regulator_Linear:AZ1117-5.0 U1
+L Regulator_Linear:AP1117-50 U1
 U 1 1 5DD7BAFC
 P 1600 6700
 F 0 "U1" H 1600 6942 50  0000 C CNN
-F 1 "AZ1117-5.0" H 1600 6851 50  0000 C CNN
-F 2 "Package_TO_SOT_SMD:SOT-223" H 1600 6950 50  0001 C CIN
+F 1 "ZLDO1117G50" H 1600 6851 50  0000 C CNN
+F 2 "Package_TO_SOT_SMD:SOT-223-3_TabPin2" H 1600 6950 50  0001 C CIN
 F 3 "~" H 1600 6700 50  0001 C CNN
 	1    1600 6700
@@
 P 5100 3700
 F 0 "U3" H 5100 4067 50  0000 C CNN
-F 1 "LM2901" H 5100 3976 50  0000 C CNN
+F 1 "LM2901D" H 5100 3976 50  0000 C CNN
 F 2 "Package_SO:SOIC-14_3.9x8.7mm_P1.27mm" H 5050 3800 50  0001 C CNN
 F 3 "~" H 5150 3900 50  0001 C CNN
